File: dboard/dboard.sch (KiCad schematic (older format))
At the start: 29 parts, among them J1 Conn_01x04, J2 Conn_01x04, U1 SRV05-4, U2 SRV05-4

Commit message: separated jlc files
Parts:
- removed C2: 470n, Capacitor_SMD:C_0805_2012Metric, symbol Device:C
- removed F2: 500mA, Fuse:Fuse_1206_3216Metric, symbol Device:Polyfuse
- removed H10, H12, H6, H8: mousebites, crokto:mousebites-6mm, symbol Mechanical:MountingHole
- removed H11, H13, H7, H9: pcba, crokto:JLCPCBA, symbol Mechanical:MountingHole
- removed H3: MountingHole, crokto:M3_Via_Hole_NC, symbol Mechanical:MountingHole
- removed H4: MountingHole_Pad, crokto:M3_Via_Hole, symbol Mechanical:MountingHole_Pad
- removed H5: jlc, crokto:jlc, symbol Mechanical:MountingHole
- removed J2: Conn_01x04, crokto:JST_SH_SM04B-SRSS-TB_1x04-1MP_P1.00mm_Horizontal, symbol Connector_Generic:Conn_01x04
- removed R4, R5: 5.1K, Resistor_SMD:R_0603_1608Metric, symbol Device:R
- removed R6: 1M, Resistor_SMD:R_1206_3216Metric, symbol Device:R
- removed U2: SRV05-4, Package_TO_SOT_SMD:SOT-23-6, symbol Power_Protection:SRV05-4
- removed USB2: HRO-TYPE-C-31-M-12, Type-C:HRO-TYPE-C-31-M-12-Assembly, symbol Type-C:HRO-TYPE-C-31-M-12
Connections:
- no-connect marks 4 -> 2

Commit message: added images
Parts:
- J1: value Conn_01x04 -> JST_SH_SM04B-SRSS-TB_1x04
Connections:
- no-connect marks 2 -> 4
Other:
- note added: "ESD & Fuse"
- note added: "JST Connector\n(not compatible with UDB)"
- note added: "Mounting Holes"
- note added: "USB Connector"
- moved on the sheet: C1, F1, H1, H2, J1, R3, U1
Changed lines of the file:
@@
 L Power_Protection:SRV05-4 U1
 U 1 1 5FEAF7BF
-P 5000 1550
-F 0 "U1" H 4550 2250 50  0000 C CNN
-F 1 "SRV05-4" H 4550 2150 50  0000 C CNN
-F 2 "Package_TO_SOT_SMD:SOT-23-6" H 5700 1100 50  0001 C CNN
-F 3 "http://www.onsemi.com/pub/Collateral/SRV05-4-D.PDF" H 5000 1550 50  0001 C CNN
-F 4 "C85364" H 5000 1550 50  0001 C CNN "jlc"
-	1    5000 1550
+P 3700 2750
+F 0 "U1" H 3250 3450 50  0000 C CNN
+F 1 "SRV05-4" H 3250 3350 50  0000 C CNN
+F 2 "Package_TO_SOT_SMD:SOT-23-6" H 4400 2300 50  0001 C CNN
+F 3 "http://www.onsemi.com/pub/Collateral/SRV05-4-D.PDF" H 3700 2750 50  0001 C CNN
+F 4 "C85364" H 3700 2750 50  0001 C CNN "jlc"
+	1    3700 2750
 	1    0    0    -1
 $EndComp
@@
 L Device:Polyfuse F1
 U 1 1 5FEB003C
-P 2750 1650
-F 0 "F1" V 2550 1650 50  0000 C CNN
-F 1 "500mA" V 2650 1650 50  0000 C CNN
-F 2 "Fuse:Fuse_1206_3216Metric" H 2800 1450 50  0001 L CNN
-F 3 "~" H 2750 1650 50  0001 C CNN
-F 4 "C70076" H 2750 1650 50  0001 C CNN "jlc"
-	1    2750 1650
+P 3700 1850
+F 0 "F1" V 3500 1850 50  0000 C CNN
+F 1 "500mA" V 3600 1850 50  0000 C CNN
+F 2 "Fuse:Fuse_1206_3216Metric" H 3750 1650 50  0001 L CNN
+F 3 "~" H 3700 1850 50  0001 C CNN
+F 4 "C70076" H 3700 1850 50  0001 C CNN "jlc"
+	1    3700 1850
 	0    1    1    0
 $EndComp
@@
 L Device:C C1
 U 1 1 5FEB0B27
-P 2300 2900
-F 0 "C1" H 2415 2946 50  0000 L CNN
-F 1 "470n" H 2415 2855 50  0000 L CNN
-F 2 "Capacitor_SMD:C_0805_2012Metric" H 2338 2750 50  0001 C CNN
-F 3 "~" H 2300 2900 50  0001 C CNN
-F 4 "C13967" H 2300 2900 50  0001 C CNN "jlc"
-	1    2300 2900
+P 2150 3200
+F 0 "C1" H 2265 3246 50  0000 L CNN
+F 1 "470n" H 2265 3155 50  0000 L CNN
+F 2 "Capacitor_SMD:C_0805_2012Metric" H 2188 3050 50  0001 C CNN
+F 3 "~" H 2150 3200 50  0001 C CNN
+F 4 "C13967" H 2150 3200 50  0001 C CNN "jlc"
+	1    2150 3200
 	1    0    0    -1
 $EndComp
@@
 L Mechanical:MountingHole_Pad H2
 U 1 1 5FEB1045
-P 4600 3050
-F 0 "H2" H 4700 3099 50  0000 L CNN
-F 1 "MountingHole_Pad" H 4700 3008 50  0000 L CNN
-F 2 "crokto:M3_Via_Hole" H 4600 3050 50  0001 C CNN
-F 3 "~" H 4600 3050 50  0001 C CNN
-	1    4600 3050
+P 4950 2450
+F 0 "H2" H 5050 2499 50  0000 L CNN
+F 1 "MountingHole_Pad" H 5050 2408 50  0000 L CNN
+F 2 "crokto:M3_Via_Hole" H 4950 2450 50  0001 C CNN
+F 3 "~" H 4950 2450 50  0001 C CNN
+	1    4950 2450
 	1    0    0    -1
 $EndComp
@@
 L Mechanical:MountingHole H1
 U 1 1 5FEB1323
-P 4600 2800
-F 0 "H1" H 4700 2846 50  0000 L CNN
-F 1 "MountingHole" H 4700 2755 50  0000 L CNN
-F 2 "crokto:M3_Via_Hole_NC" H 4600 2800 50  0001 C CNN
-F 3 "~" H 4600 2800 50  0001 C CNN
-	1    4600 2800
+P 4950 2200
+F 0 "H1" H 5050 2246 50  0000 L CNN
+F 1 "MountingHole" H 5050 2155 50  0000 L CNN
+F 2 "crokto:M3_Via_Hole_NC" H 4950 2200 50  0001 C CNN
+F 3 "~" H 4950 2200 50  0001 C CNN
+	1    4950 2200
 	1    0    0    -1
 $EndComp
@@
 L Device:R R3
 U 1 1 5FEB31E8
-P 2000 2900
-F 0 "R3" H 2070 2946 50  0000 L CNN
-F 1 "1M" H 2070 2855 50  0000 L CNN
-F 2 "Resistor_SMD:R_1206_3216Metric" V 1930 2900 50  0001 C CNN
-F 3 "~" H 2000 2900 50  0001 C CNN
-F 4 "C17927" H 2000 2900 50  0001 C CNN "jlc"
-	1    2000 2900
+P 1850 3200
+F 0 "R3" H 1920 3246 50  0000 L CNN
+F 1 "1M" H 1920 3155 50  0000 L CNN
+F 2 "Resistor_SMD:R_1206_3216Metric" V 1780 3200 50  0001 C CNN
+F 3 "~" H 1850 3200 50  0001 C CNN
+F 4 "C17927" H 1850 3200 50  0001 C CNN "jlc"
+	1    1850 3200
 	1    0    0    -1
 $EndComp
@@
 $EndComp
 Wire Wire Line
-	2600 1650 2400 1650
-Connection ~ 2400 1650
-Wire Wire Line
 	2400 1650 2000 1650
-Text GLabel 5500 1450 2    50   Input ~ 0
+Text GLabel 4200 2650 2    50   Input ~ 0
 D+
-Text GLabel 4500 1650 0    50   Input ~ 0
+Text GLabel 3200 2850 0    50   Input ~ 0
 D-
 Wire Wire Line
@@
 $EndComp
 Wire Wire Line
-	2000 2750 2300 2750
-Connection ~ 2000 2750
-Wire Wire Line
-	2000 3050 2300 3050
-Text GLabel 2300 2750 2    50   Input ~ 0
+	1850 3350 2150 3350
+Text GLabel 2000 2750 2    50   Input ~ 0
 SHIELD
 $Comp
 L power:GND #PWR010
 U 1 1 5FEBE302
-P 2000 3050
-F 0 "#PWR010" H 2000 2800 50  0001 C CNN
-F 1 "GND" H 2005 2877 50  0000 C CNN
-F 2 "" H 2000 3050 50  0001 C CNN
-F 3 "" H 2000 3050 50  0001 C CNN
-	1    2000 3050
-	1    0    0    -1
-$EndComp
-Connection ~ 2000 3050
+P 1850 3350
+F 0 "#PWR010" H 1850 3100 50  0001 C CNN
+F 1 "GND" H 1855 3177 50  0000 C CNN
+F 2 "" H 1850 3350 50  0001 C CNN
+F 3 "" H 1850 3350 50  0001 C CNN
+	1    1850 3350
+	1    0    0    -1
+$EndComp
+Connection ~ 1850 3350
 $Comp
 L power:+5V #PWR04
 U 1 1 5FEBEA41
-P 2900 1650
-F 0 "#PWR04" H 2900 1500 50  0001 C CNN
-F 1 "+5V" V 2915 1778 50  0000 L CNN
-F 2 "" H 2900 1650 50  0001 C CNN
-F 3 "" H 2900 1650 50  0001 C CNN
-	1    2900 1650
-	0    1    1    0
+P 3950 1850
+F 0 "#PWR04" H 3950 1700 50  0001 C CNN
+F 1 "+5V" V 3965 1978 50  0000 L CNN
+F 2 "" H 3950 1850 50  0001 C CNN
+F 3 "" H 3950 1850 50  0001 C CNN
+	1    3950 1850
+	1    0    0    -1
 $EndComp
 $Comp
 L power:+5V #PWR01
 U 1 1 5FEBF8CE
-P 5000 1050
-F 0 "#PWR01" H 5000 900 50  0001 C CNN
-F 1 "+5V" H 5015 1223 50  0000 C CNN
-F 2 "" H 5000 1050 50  0001 C CNN
-F 3 "" H 5000 1050 50  0001 C CNN
-	1    5000 1050
+P 3700 2250
+F 0 "#PWR01" H 3700 2100 50  0001 C CNN
+F 1 "+5V" H 3715 2423 50  0000 C CNN
+F 2 "" H 3700 2250 50  0001 C CNN
+F 3 "" H 3700 2250 50  0001 C CNN
+	1    3700 2250
 	1    0    0    -1
 $EndComp
@@
 L power:GND #PWR06
 U 1 1 5FEC0294
-P 5000 2050
-F 0 "#PWR06" H 5000 1800 50  0001 C CNN
-F 1 "GND" H 5005 1877 50  0000 C CNN
-F 2 "" H 5000 2050 50  0001 C CNN
-F 3 "" H 5000 2050 50  0001 C CNN
-	1    5000 2050
-	1    0    0    -1
-$EndComp
-Text GLabel 4600 3150 3    50   Input ~ 0
+P 3700 3250
+F 0 "#PWR06" H 3700 3000 50  0001 C CNN
+F 1 "GND" H 3705 3077 50  0000 C CNN
+F 2 "" H 3700 3250 50  0001 C CNN
+F 3 "" H 3700 3250 50  0001 C CNN
+	1    3700 3250
+	1    0    0    -1
+$EndComp
+Text GLabel 4950 2550 3    50   Input ~ 0
 SHIELD
+Text GLabel 2100 1950 2    50   Input ~ 0
+D-
+Text GLabel 2250 2050 2    50   Input ~ 0
+D+
+NoConn ~ 3200 2650
+NoConn ~ 4200 2850
+Wire Wire Line
+	2200 2050 2250 2050
+Connection ~ 2200 2050
+$Comp
+L power:VBUS #PWR?
+U 1 1 6002061A
+P 3450 1850
+F 0 "#PWR?" H 3450 1700 50  0001 C CNN
+F 1 "VBUS" H 3465 2023 50  0000 C CNN
+F 2 "" H 3450 1850 50  0001 C CNN
+F 3 "" H 3450 1850 50  0001 C CNN
+	1    3450 1850
+	1    0    0    -1
+$EndComp
+Wire Wire Line
+	3550 1850 3450 1850
+Wire Wire Line
+	3950 1850 3850 1850
+Wire Wire Line
+	2150 3050 1850 3050
+Text GLabel 1750 3050 0    50   Input ~ 0
+SHIELD
+Wire Wire Line
+	1750 3050 1850 3050
+Connection ~ 1850 3050
 $Comp
 L Connector_Generic:Conn_01x04 J1
 U 1 1 5FEC6F34
-P 6950 2750
-F 0 "J1" H 7030 2742 50  0000 L CNN
-F 1 "Conn_01x04" H 7030 2651 50  0000 L CNN
-F 2 "crokto:JST_SH_SM04B-SRSS-TB_1x04-1MP_P1.00mm_Horizontal" H 6950 2750 50  0001 C CNN
-F 3 "~" H 6950 2750 50  0001 C CNN
-	1    6950 2750
+P 6600 2300
+F 0 "J1" V 6850 2250 50  0000 C CNN
+F 1 "JST_SH_SM04B-SRSS-TB_1x04" V 6750 2250 50  0000 C CNN
+F 2 "crokto:JST_SH_SM04B-SRSS-TB_1x04-1MP_P1.00mm_Horizontal" H 6600 2300 50  0001 C CNN
+F 3 "~" H 6600 2300 50  0001 C CNN
+	1    6600 2300
 	1    0    0    -1
 $EndComp
@@
 L power:GND #PWR0101
 U 1 1 5FEC7655
-P 6750 2950
-F 0 "#PWR0101" H 6750 2700 50  0001 C CNN
-F 1 "GND" H 6755 2777 50  0000 C CNN
-F 2 "" H 6750 2950 50  0001 C CNN
-F 3 "" H 6750 2950 50  0001 C CNN
-	1    6750 2950
+P 6400 2500
+F 0 "#PWR0101" H 6400 2250 50  0001 C CNN
+F 1 "GND" H 6405 2327 50  0000 C CNN
+F 2 "" H 6400 2500 50  0001 C CNN
+F 3 "" H 6400 2500 50  0001 C CNN
+	1    6400 2500
 	1    0    0    -1
 $EndComp
@@
 L power:+5V #PWR0102
 U 1 1 5FEC7B14
-P 6750 2650
-F 0 "#PWR0102" H 6750 2500 50  0001 C CNN
-F 1 "+5V" H 6765 2823 50  0000 C CNN
-F 2 "" H 6750 2650 50  0001 C CNN
-F 3 "" H 6750 2650 50  0001 C CNN
-	1    6750 2650
-	1    0    0    -1
-$EndComp
-Text GLabel 6750 2750 0    50   Input ~ 0
+P 6400 2200
+F 0 "#PWR0102" H 6400 2050 50  0001 C CNN
+F 1 "+5V" H 6415 2373 50  0000 C CNN
+F 2 "" H 6400 2200 50  0001 C CNN
+F 3 "" H 6400 2200 50  0001 C CNN
+	1    6400 2200
+	1    0    0    -1
+$EndComp
+Text GLabel 6400 2300 0    50   Input ~ 0
 D+
-Text GLabel 6750 2850 0    50   Input ~ 0
+Text GLabel 6400 2400 0    50   Input ~ 0
 D-
-Text GLabel 2100 1950 2    50   Input ~ 0
-D-
-Text GLabel 2200 2050 2    50   Input ~ 0
-D+
+Text Notes 1500 3700 0    50   ~ 0
+USB Connector
+Text Notes 3500 3700 0    50   ~ 0
+ESD & Fuse
+Text Notes 4950 3700 0    50   ~ 0
+Mounting Holes
+Text Notes 6200 3700 0    50   ~ 0
+JST Connector\n(not compatible with UDB)
 $EndSCHEMATC

Commit message: a bunch of new dboards
Parts:
- added D1: D_TVS, Diode_SMD:D_SOD-123F, symbol Device:D_TVS
- J1: jlc (none) -> C160404
- USB1: value HRO-TYPE-C-31-M-12 -> HRO-TYPE-C-31-M-14; footprint Type-C:HRO-TYPE-C-31-M-12-Assembly -> Type-C:HRO-TYPE-C-31-M-14
Other:
- moved on the sheet: J1
Changed lines of the file:
@@
 P 1900 2100
 F 0 "USB1" V 1200 2100 60  0000 C CNN
-F 1 "HRO-TYPE-C-31-M-12" V 1300 2100 60  0000 C CNN
-F 2 "Type-C:HRO-TYPE-C-31-M-12-Assembly" H 1900 2100 60  0001 C CNN
+F 1 "HRO-TYPE-C-31-M-14" V 1300 2100 60  0000 C CNN
+F 2 "Type-C:HRO-TYPE-C-31-M-14" H 1900 2100 60  0001 C CNN
 F 3 "" H 1900 2100 60  0001 C CNN
 	1    1900 2100
@@
 Wire Wire Line
 	2400 1650 2000 1650
+Text GLabel 3200 2850 0    50   Input ~ 0
+D+
 Text GLabel 4200 2650 2    50   Input ~ 0
-D+
-Text GLabel 3200 2850 0    50   Input ~ 0
 D-
 Wire Wire Line
@@
 Connection ~ 2200 2050
 $Comp
-L power:VBUS #PWR?
+L power:VBUS #PWR0103
 U 1 1 6002061A
 P 3450 1850
-F 0 "#PWR?" H 3450 1700 50  0001 C CNN
+F 0 "#PWR0103" H 3450 1700 50  0001 C CNN
 F 1 "VBUS" H 3465 2023 50  0000 C CNN
 F 2 "" H 3450 1850 50  0001 C CNN
@@
 L Connector_Generic:Conn_01x04 J1
 U 1 1 5FEC6F34
-P 6600 2300
-F 0 "J1" V 6850 2250 50  0000 C CNN
-F 1 "JST_SH_SM04B-SRSS-TB_1x04" V 6750 2250 50  0000 C CNN
-F 2 "crokto:JST_SH_SM04B-SRSS-TB_1x04-1MP_P1.00mm_Horizontal" H 6600 2300 50  0001 C CNN
-F 3 "~" H 6600 2300 50  0001 C CNN
-	1    6600 2300
+P 6600 2350
+F 0 "J1" V 6850 2300 50  0000 C CNN
+F 1 "JST_SH_SM04B-SRSS-TB_1x04" V 6750 2300 50  0000 C CNN
+F 2 "crokto:JST_SH_SM04B-SRSS-TB_1x04-1MP_P1.00mm_Horizontal" H 6600 2350 50  0001 C CNN
+F 3 "~" H 6600 2350 50  0001 C CNN
+F 4 "C160404" H 6600 2350 50  0001 C CNN "jlc"
+	1    6600 2350
 	1    0    0    -1
 $EndComp
@@
 L power:GND #PWR0101
 U 1 1 5FEC7655
-P 6400 2500
-F 0 "#PWR0101" H 6400 2250 50  0001 C CNN
-F 1 "GND" H 6405 2327 50  0000 C CNN
-F 2 "" H 6400 2500 50  0001 C CNN
-F 3 "" H 6400 2500 50  0001 C CNN
-	1    6400 2500
+P 6400 2550
+F 0 "#PWR0101" H 6400 2300 50  0001 C CNN
+F 1 "GND" H 6405 2377 50  0000 C CNN
+F 2 "" H 6400 2550 50  0001 C CNN
+F 3 "" H 6400 2550 50  0001 C CNN
+	1    6400 2550
 	1    0    0    -1
 $EndComp
@@
 L power:+5V #PWR0102
 U 1 1 5FEC7B14
-P 6400 2200
-F 0 "#PWR0102" H 6400 2050 50  0001 C CNN
-F 1 "+5V" H 6415 2373 50  0000 C CNN
-F 2 "" H 6400 2200 50  0001 C CNN
-F 3 "" H 6400 2200 50  0001 C CNN
-	1    6400 2200
-	1    0    0    -1
-$EndComp
-Text GLabel 6400 2300 0    50   Input ~ 0
+P 6400 2250
+F 0 "#PWR0102" H 6400 2100 50  0001 C CNN
+F 1 "+5V" H 6415 2423 50  0000 C CNN
+F 2 "" H 6400 2250 50  0001 C CNN
+F 3 "" H 6400 2250 50  0001 C CNN
+	1    6400 2250
+	1    0    0    -1
+$EndComp
+Text GLabel 6400 2450 0    50   Input ~ 0
 D+
-Text GLabel 6400 2400 0    50   Input ~ 0
+Text GLabel 6400 2350 0    50   Input ~ 0
 D-
 Text Notes 1500 3700 0    50   ~ 0
@@
 Text Notes 6200 3700 0    50   ~ 0
 JST Connector\n(not compatible with UDB)
+$Comp
+L power:+5V #PWR0104
+U 1 1 60467AC3
+P 3550 1250
+F 0 "#PWR0104" H 3550 1100 50  0001 C CNN
+F 1 "+5V" H 3565 1423 50  0000 C CNN
+F 2 "" H 3550 1250 50  0001 C CNN
+F 3 "" H 3550 1250 50  0001 C CNN
+	1    3550 1250
+	1    0    0    -1
+$EndComp
+$Comp
+L power:GND #PWR0105
+U 1 1 60468083
+P 3850 1250
+F 0 "#PWR0105" H 3850 1000 50  0001 C CNN
+F 1 "GND" H 3855 1077 50  0000 C CNN
+F 2 "" H 3850 1250 50  0001 C CNN
+F 3 "" H 3850 1250 50  0001 C CNN
+	1    3850 1250
+	1    0    0    -1
+$EndComp
+$Comp
+L Device:D_TVS D1
+U 1 1 604674B7
+P 3700 1250
+F 0 "D1" H 3700 1467 50  0000 C CNN
+F 1 "D_TVS" H 3700 1376 50  0000 C CNN
+F 2 "Diode_SMD:D_SOD-123F" H 3700 1250 50  0001 C CNN
+F 3 "~" H 3700 1250 50  0001 C CNN
+F 4 "C78395" H 3700 1250 50  0001 C CNN "jlc"
+	1    3700 1250
+	1    0    0    -1
+$EndComp
 $EndSCHEMATC
